File: JellyLoad-Combi_V2-0/JellyLoad-Combi_V2-0.kicad_sch (KiCad schematic)
At the start: 26 parts, among them J1 Conn_02x07_Odd_Even, Q1 SFH3710-4, Q2 SFH3710-4, Q3 SFH3710-4, Q4 SFH3710-4, Q5 SFH3710-4, Q6 SFH3710-4, Q7 SFH3710-4, Q8 SFH3710-4, Q9 SFH3710-4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

Commit message: Admin updates to schematic and layout
Parts:
- Q1, Q2, Q3, Q4, Q5, Q6, Q7, Q8, Q9: footprint OptoDevice:Osram_SFH3710-4 -> OptoDevice:Osram_SFH3710
Other:
- moved on the sheet: D1, D2, J1, Q1, Q2, Q3, Q4, Q5, Q6, Q7, Q8, Q9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

Commit message: Update to BOM
LED part numbers changed to be RED LED consistently with JLC and Digikey
Parts:
- D1: JLC PN C19273151 -> C19171390
Changed lines of the file:
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@@
 			)
 		)
-		(property "JLC PN" "C19273151"
+		(property "JLC PN" "C19171390"
 			(at 251.46 64.77 90)
 			(effects
